Commit message: fix wheelDiameter

File: mega3_description/urdf/mega3.xacro (robot description, xacro)
@@ -34,5 +34,5 @@
 <link name="left_wheel_1">
   <inertial>
-    <origin xyz="0.0 0.0 0.03313" rpy="0 1.5708 0"/>
+    <origin xyz="0.0 0.0 0.00213" rpy="0 1.5708 0"/>
     <mass value="1.239934"/>
     <inertia ixx="0.002474" iyy="0.00174" izz="0.00174"
@@ -41,5 +41,5 @@
   </inertial>
   <visual>
-    <origin xyz="-0.07 -0.1 -0.105" rpy="0 1.5708 0"/>
+    <origin xyz="-0.07 -0.1 -0.136" rpy="0 1.5708 0"/>
     <geometry>
       <mesh filename="package://mega3_description/meshes/left_wheel_1.stl" scale="0.001 0.001 0.001"/>
@@ -56,5 +56,5 @@
 <link name="right_wheel_1">
   <inertial>
-    <origin xyz="0 0 -0.03313" rpy="0 1.5708 0"/>
+    <origin xyz="0 0 -0.00213" rpy="0 1.5708 0"/>
     <mass value="1.239934"/>
     <inertia ixx="0.002474" iyy="0.00174" izz="0.00174"
@@ -63,5 +63,5 @@
   </inertial>
   <visual>
-    <origin xyz="-0.07 -0.1 0.105" rpy="0 1.5708 0"/>
+    <origin xyz="-0.07 -0.1 0.136" rpy="0 1.5708 0"/>
     <geometry>
       <mesh filename="package://mega3_description/meshes/right_wheel_1.stl" scale="0.001 0.001 0.001"/>
@@ -77,5 +77,5 @@
 </link>
 <joint name="left_wheel_joint" type="continuous">
-  <origin xyz="-0.105 0.1 0.07" rpy="0 -1.5708 0"/>
+  <origin xyz="-0.136 0.1 0.07" rpy="0 -1.5708 0"/>
   <parent link="base_link"/>
   <child link="left_wheel_1"/>
@@ -83,5 +83,5 @@
 </joint>
 <joint name="right_wheel_joint" type="continuous">
-  <origin xyz="0.105 0.1 0.07" rpy="0 -1.5708 0"/>
+  <origin xyz="0.136 0.1 0.07" rpy="0 -1.5708 0"/>
   <parent link="base_link"/>
   <child link="right_wheel_1"/>

Commit message: fix collision origin

File: mega3_description/urdf/mega3.xacro (robot description, xacro)
@@ -48,5 +48,5 @@
   </visual>
   <collision>
-    <origin xyz="-0.07 -0.1 -0.105" rpy="0 1.5708 0"/>
+    <origin xyz="-0.07 -0.1 -0.136" rpy="0 1.5708 0"/>
     <geometry>
       <mesh filename="package://mega3_description/meshes/left_wheel_1.stl" scale="0.001 0.001 0.001"/>
@@ -70,5 +70,5 @@
   </visual>
   <collision>
-    <origin xyz="-0.07 -0.1 0.105" rpy="0 1.5708 0"/>
+    <origin xyz="-0.07 -0.1 0.136" rpy="0 1.5708 0"/>
     <geometry>
       <mesh filename="package://mega3_description/meshes/right_wheel_1.stl" scale="0.001 0.001 0.001"/>
