Commit message: Use native Jazzy Harmonic model definitions and updated caster meshes

File: urdf/f120a.xacro (robot description, xacro)
@@ -1,7 +1,9 @@
 <?xml version="1.0"?>
 <robot name="f120a" xmlns:xacro="http://www.ros.org/wiki/xacro">
+  <xacro:arg name="use_ros2_control" default="true" />
+  <xacro:arg name="lidar" default="true" />
+  <xacro:property name="tg30_enabled" value="false" />
   <xacro:include filename="$(find megarover_description)/urdf/materials.xacro" />
   <xacro:include filename="$(find megarover_description)/urdf/f120a.gazebo" />
-  <xacro:arg name="use_ros2_control" default="true" />
   <xacro:if value="$(arg use_ros2_control)">
     <xacro:include filename="$(find megarover_description)/urdf/f120a_ros2_control.xacro" />
@@ -34,12 +36,12 @@
   <link name="base_link">
     <inertial>
-      <origin xyz="-0.012552 0.000002 0.124849" rpy="0 0 0" />
-      <mass value="26.5" />
-      <inertia ixx="2.862913e-01" iyy="3.703059e-01" izz="5.773479e-01"
-        ixy="-1.109256e-05" iyz="8.886529e-07"
-        ixz="4.327049e-03" />
+      <origin xyz="-0.013369162863708595 0.003967105997105071 0.13087762523743113" rpy="0 0 0" />
+      <mass value="6.991126256639111" />
+      <inertia ixx="0.10171936472593801" iyy="0.12309534845763971" izz="0.1862309757885538"
+        ixy="-3.9446830044943695e-05" iyz="0.00020498239448746465"
+        ixz="0.012608115312944097" />
     </inertial>
     <visual>
-      <origin xyz="0 0 0" rpy="0 0 -1.5708" />
+      <origin xyz="0 0 0" rpy="0 0 0" />
       <geometry>
         <mesh filename="package://megarover_description/meshes/f120a/base_link.stl" scale="0.001 0.001 0.001" />
@@ -48,7 +50,91 @@
     </visual>
     <collision>
-      <origin xyz="0 0 0" rpy="0 0 -1.5708" />
+      <origin xyz="0 0 0" rpy="0 0 0" />
       <geometry>
         <mesh filename="package://megarover_description/meshes/f120a/base_link.stl" scale="0.001 0.001 0.001" />
+      </geometry>
+    </collision>
+  </link>
+  <joint name="battery_joint" type="fixed">
+    <origin xyz="0.0 0.005 0.0" rpy="0 0 0" />
+    <parent link="base_link" />
+    <child link="Battery" />
+  </joint>
+  <link name="Battery">
+    <inertial>
+      <origin xyz="-0.00047690262730757597 -1.214306433183765e-17 0.12084712924012407" rpy="0 0 0" />
+      <mass value="14.366266000000003" />
+      <inertia ixx="0.149967155276439" iyy="0.05463969367969923" izz="0.16733910801756052"
+        ixy="4.588208068687094e-17" iyz="2.2551405187698492e-17" ixz="0.0003847207249658767" />
+    </inertial>
+    <visual>
+      <origin xyz="0.0 -0.005 0.0" rpy="0 0 0" />
+      <geometry>
+        <mesh filename="package://megarover_description/meshes/f120a/Battery.stl" scale="0.001 0.001 0.001" />
+      </geometry>
+      <material name="silver" />
+    </visual>
+    <collision>
+      <origin xyz="0.0 -0.005 0.0" rpy="0 0 0" />
+      <geometry>
+        <mesh filename="package://megarover_description/meshes/f120a/Battery.stl" scale="0.001 0.001 0.001" />
+      </geometry>
+    </collision>
+  </link>
+  <joint name="caster_swivel_joint" type="continuous">
+    <origin xyz="-0.185 0.005 0.141" rpy="0 0 0" />
+    <parent link="base_link" />
+    <child link="Caster_Frame" />
+    <axis xyz="0.0 0.0 1.0" />
+    <limit effort="100.0" velocity="100.0" />
+  </joint>
+  <link name="Caster_Frame">
+    <inertial>
+      <origin xyz="-0.007262242104825234 -1.734723475976807e-16 -0.01913205916374887" rpy="0 0 0" />
+      <mass value="0.2102704532022103" />
+      <inertia ixx="0.00016899802664020747" iyy="0.00020027057626632871" izz="0.0001547263035165296"
+        ixy="3.2526065174565133e-19" iyz="-1.463672932855431e-18" ixz="-5.075055445010607e-05" />
+    </inertial>
+    <visual>
+      <origin xyz="0.185 -0.005 -0.141" rpy="0 0 0" />
+      <geometry>
+        <mesh filename="package://megarover_description/meshes/f120a/Caster_Frame.stl" scale="0.001 0.001 0.001" />
+      </geometry>
+      <material name="silver" />
+    </visual>
+    <collision>
+      <origin xyz="0.185 -0.005 -0.141" rpy="0 0 0" />
+      <geometry>
+        <mesh filename="package://megarover_description/meshes/f120a/Caster_Frame.stl" scale="0.001 0.001 0.001" />
+      </geometry>
+    </collision>
+  </link>
+  <joint name="caster_wheel_joint" type="continuous">
+    <origin xyz="-0.04 -0.0205 -0.091" rpy="0 0 0" />
+    <parent link="Caster_Frame" />
+    <child link="Caster_Wheel" />
+    <axis xyz="0.0 -1.0 0.0" />
+    <limit effort="100.0" velocity="100.0" />
+  </joint>
+  <link name="Caster_Wheel">
+    <inertial>
+      <origin xyz="2.7755575615628914e-17 0.02049999999999995 6.938893903907228e-18" rpy="0 0 0" />
+      <mass value="0.2913827186204193" />
+      <inertia ixx="0.00021185951833023898" iyy="0.00036422839827547626" izz="0.00021185951833024332"
+        ixy="2.168404344971009e-19" iyz="1.8973538018496328e-19" ixz="-3.0357660829594124e-18" />
+    </inertial>
+    <visual>
+      <origin xyz="0.225 0.0155 -0.05" rpy="0 0 0" />
+      <geometry>
+        <mesh filename="package://megarover_description/meshes/f120a/Caster_Wheel.stl" scale="0.001 0.001 0.001" />
+      </geometry>
+      <material name="caster_wheel">
+        <color rgba="0.960784 0.960784 0.952941 1" />
+      </material>
+    </visual>
+    <collision>
+      <origin xyz="0.225 0.0155 -0.05" rpy="0 0 0" />
+      <geometry>
+        <mesh filename="package://megarover_description/meshes/f120a/Caster_Wheel.stl" scale="0.001 0.001 0.001" />
       </geometry>
     </collision>
@@ -69,5 +155,5 @@
     </inertial>
     <visual>
-      <origin xyz="-0.108 0.202 -0.085" rpy="0 0 -1.5708" />
+      <origin xyz="-0.108 0.197 -0.085" rpy="0 0 0" />
       <geometry>
         <mesh filename="package://megarover_description/meshes/f120a/right_wheel_1.stl" scale="0.001 0.001 0.001" />
@@ -76,7 +162,7 @@
     </visual>
     <collision>
-      <origin xyz="0 0 0" rpy="1.5708 0 0" />
+      <origin xyz="-0.108 0.197 -0.085" rpy="0 0 0" />
       <geometry>
-        <cylinder radius="0.085" length="0.05" />
+        <mesh filename="package://megarover_description/meshes/f120a/right_wheel_1.stl" scale="0.001 0.001 0.001" />
       </geometry>
     </collision>
@@ -97,5 +183,5 @@
     </inertial>
     <visual>
-      <origin xyz="-0.108 -0.202 -0.085" rpy="0 0 -1.5708" />
+      <origin xyz="-0.108297 -0.202941 -0.087693" rpy="0 0 0" />
       <geometry>
         <mesh filename="package://megarover_description/meshes/f120a/left_wheel_1.stl" scale="0.001 0.001 0.001" />
@@ -104,9 +190,10 @@
     </visual>
     <collision>
-      <origin xyz="0 0 0" rpy="1.5708 0 0" />
+      <origin xyz="-0.108297 -0.202941 -0.087693" rpy="0 0 0" />
       <geometry>
-        <cylinder radius="0.085" length="0.05" />
+        <mesh filename="package://megarover_description/meshes/f120a/left_wheel_1.stl" scale="0.001 0.001 0.001" />
       </geometry>
     </collision>
   </link>
+  <xacro:gazebo_sensors />
 </robot>

File: urdf/f120a_ros2_control.xacro (robot description, xacro)
@@ -3,5 +3,5 @@
   <ros2_control name="GazeboSystem" type="system">
     <hardware>
-      <plugin>gazebo_ros2_control/GazeboSystem</plugin>
+      <plugin>gz_ros2_control/GazeboSimSystem</plugin>
     </hardware>
     <joint name="left_wheel_joint">
@@ -15,4 +15,12 @@
       <state_interface   name="position"/>
     </joint>
+    <joint name="caster_swivel_joint">
+      <state_interface name="velocity"/>
+      <state_interface name="position"/>
+    </joint>
+    <joint name="caster_wheel_joint">
+      <state_interface name="velocity"/>
+      <state_interface name="position"/>
+    </joint>
   </ros2_control>
 </robot>

File: urdf/mega3.xacro (robot description, xacro)
@@ -1,7 +1,9 @@
 <?xml version="1.0"?>
 <robot name="mega3" xmlns:xacro="http://www.ros.org/wiki/xacro">
+  <xacro:arg name="use_ros2_control" default="true" />
+  <xacro:arg name="lidar" default="true" />
+  <xacro:property name="tg30_enabled" value="false" />
   <xacro:include filename="$(find megarover_description)/urdf/materials.xacro" />
   <xacro:include filename="$(find megarover_description)/urdf/mega3.gazebo" />
-  <xacro:arg name="use_ros2_control" default="true" />
   <xacro:if value="$(arg use_ros2_control)">
     <xacro:include filename="$(find megarover_description)/urdf/mega3_ros2_control.xacro" />
@@ -34,9 +36,9 @@
   <link name="base_link">
     <inertial>
-      <origin xyz="-0.000007 -0.000146 0.095171" rpy="0 0 0" />
-      <mass value="12" />
-      <inertia ixx="5.644759e-02" iyy="9.308603e-02" izz="1.250700e-01"
-        ixy="-3.125032e-04" iyz="-2.117978e-05"
-        ixz="-2.464583e-03" />
+      <origin xyz="0.008652929776791014 0.001107013730491935 0.10307586165229349" rpy="0 0 -1.5707963267948966" />
+      <mass value="3.2472141930264886" />
+      <inertia ixx="0.03499380367357023" iyy="0.02389566038235242" izz="0.04961607321095147"
+        ixy="0.0004073496120585377" iyz="-0.0008864404421181438"
+        ixz="5.121736313081106e-05" />
     </inertial>
     <visual>
@@ -51,4 +53,89 @@
       <geometry>
         <mesh filename="package://megarover_description/meshes/mega3/base_link.stl" scale="0.001 0.001 0.001" />
+      </geometry>
+    </collision>
+  </link>
+  <!-- CAD +Y forward is rotated into the existing mega3 +X frame. -->
+  <joint name="battery_joint" type="fixed">
+    <origin xyz="0 0 0" rpy="0 0 -1.5707963267948966" />
+    <parent link="base_link" />
+    <child link="Battery" />
+  </joint>
+  <link name="Battery">
+    <inertial>
+      <origin xyz="-8.617707998157631e-18 0.008998698470897024 0.08943706012717803" rpy="0 0 0" />
+      <mass value="8.245147502236165" />
+      <inertia ixx="0.0214853104155929" iyy="0.03313493288601588" izz="0.04284993321973867"
+        ixy="-7.034280604820041e-18" iyz="4.959248083875184e-07" ixz="-6.705434520297627e-19" />
+    </inertial>
+    <visual>
+      <origin xyz="0 0 0" rpy="0 0 0" />
+      <geometry>
+        <mesh filename="package://megarover_description/meshes/mega3/Battery.stl" scale="0.001 0.001 0.001" />
+      </geometry>
+      <material name="silver" />
+    </visual>
+    <collision>
+      <origin xyz="0 0 0" rpy="0 0 0" />
+      <geometry>
+        <mesh filename="package://megarover_description/meshes/mega3/Battery.stl" scale="0.001 0.001 0.001" />
+      </geometry>
+    </collision>
+  </link>
+  <joint name="caster_swivel_joint" type="continuous">
+    <origin xyz="-0.13 0 0.0814" rpy="0 0 -1.5707963267948966" />
+    <parent link="base_link" />
+    <child link="Caster_Frame" />
+    <axis xyz="0 0 -1" />
+    <limit effort="100.0" velocity="100.0" />
+  </joint>
+  <link name="Caster_Frame">
+    <inertial>
+      <origin xyz="-2.9997809438943724e-18 0.0008380877975086853 -0.019114933984371356" rpy="0 0 0" />
+      <mass value="0.18593892620957955" />
+      <inertia ixx="4.784843078569148e-05" iyy="4.884288359081478e-05" izz="3.484845036761698e-05"
+        ixy="-3.951178862922994e-20" iyz="-4.376302309193466e-06" ixz="-3.4741117944938427e-20" />
+    </inertial>
+    <visual>
+      <origin xyz="0 0.13 -0.0814" rpy="0 0 0" />
+      <geometry>
+        <mesh filename="package://megarover_description/meshes/mega3/Caster_Frame.stl" scale="0.001 0.001 0.001" />
+      </geometry>
+      <material name="silver" />
+    </visual>
+    <collision>
+      <origin xyz="0 0.13 -0.0814" rpy="0 0 0" />
+      <geometry>
+        <mesh filename="package://megarover_description/meshes/mega3/Caster_Frame.stl" scale="0.001 0.001 0.001" />
+      </geometry>
+    </collision>
+  </link>
+  <joint name="caster_wheel_joint" type="continuous">
+    <origin xyz="0.014 -0.021 -0.0489" rpy="0 0 0" />
+    <parent link="Caster_Frame" />
+    <child link="Caster_Wheel" />
+    <axis xyz="1 0 0" />
+    <limit effort="100.0" velocity="100.0" />
+  </joint>
+  <link name="Caster_Wheel">
+    <inertial>
+      <origin xyz="-0.014 2.7755575615628914e-17 0.0" rpy="0 0 0" />
+      <mass value="0.07034811349550506" />
+      <inertia ixx="3.7152597439811096e-05" iyy="2.092123583642218e-05" izz="2.0921235836423007e-05"
+        ixy="9.038103598868473e-21" iyz="-3.2526065174565133e-19" ixz="0.0" />
+    </inertial>
+    <visual>
+      <origin xyz="-0.014 0.151 -0.0325" rpy="0 0 0" />
+      <geometry>
+        <mesh filename="package://megarover_description/meshes/mega3/Caster_Wheel.stl" scale="0.001 0.001 0.001" />
+      </geometry>
+      <material name="caster_wheel">
+        <color rgba="0.960784 0.960784 0.952941 1" />
+      </material>
+    </visual>
+    <collision>
+      <origin xyz="-0.014 0.151 -0.0325" rpy="0 0 0" />
+      <geometry>
+        <mesh filename="package://megarover_description/meshes/mega3/Caster_Wheel.stl" scale="0.001 0.001 0.001" />
       </geometry>
     </collision>
@@ -76,7 +163,7 @@
     </visual>
     <collision>
-      <origin xyz="0 0 0" rpy="-1.5708 0 0" />
-      <geometry>
-        <cylinder radius="0.07" length="0.05" />
+      <origin xyz="-0.1 -0.136 -0.07" rpy="0 0 -1.5708" />
+      <geometry>
+        <mesh filename="package://megarover_description/meshes/mega3/left_wheel_1.stl" scale="0.001 0.001 0.001" />
       </geometry>
     </collision>
@@ -104,9 +191,10 @@
     </visual>
     <collision>
-      <origin xyz="0 0 0" rpy="-1.5708 0 0" />
-      <geometry>
-        <cylinder radius="0.07" length="0.05" />
-      </geometry>
-    </collision>
-  </link>
+      <origin xyz="-0.1 0.136 -0.07" rpy="0 0 -1.5708" />
+      <geometry>
+        <mesh filename="package://megarover_description/meshes/mega3/right_wheel_1.stl" scale="0.001 0.001 0.001" />
+      </geometry>
+    </collision>
+  </link>
+  <xacro:gazebo_sensors />
 </robot>

File: urdf/mega3_ros2_control.xacro (robot description, xacro)
@@ -3,5 +3,5 @@
   <ros2_control name="GazeboSystem" type="system">
     <hardware>
-      <plugin>gazebo_ros2_control/GazeboSystem</plugin>
+      <plugin>gz_ros2_control/GazeboSimSystem</plugin>
     </hardware>
     <joint name="left_wheel_joint">
@@ -15,4 +15,12 @@
       <state_interface   name="position"/>
     </joint>
+    <joint name="caster_swivel_joint">
+      <state_interface name="velocity"/>
+      <state_interface name="position"/>
+    </joint>
+    <joint name="caster_wheel_joint">
+      <state_interface name="velocity"/>
+      <state_interface name="position"/>
+    </joint>
   </ros2_control>
 </robot>

File: urdf/s40a_lb.xacro (robot description, xacro)
@@ -1,7 +1,9 @@
 <?xml version="1.0"?>
 <robot name="s40a_lb" xmlns:xacro="http://www.ros.org/wiki/xacro">
+  <xacro:arg name="use_ros2_control" default="true" />
+  <xacro:arg name="lidar" default="true" />
+  <xacro:property name="tg30_enabled" value="false" />
   <xacro:include filename="$(find megarover_description)/urdf/materials.xacro" />
   <xacro:include filename="$(find megarover_description)/urdf/s40a_lb.gazebo" />
-  <xacro:arg name="use_ros2_control" default="true" />
   <xacro:if value="$(arg use_ros2_control)">
     <xacro:include filename="$(find megarover_description)/urdf/s40a_lb_ros2_control.xacro" />
@@ -363,12 +365,13 @@
     child="back_left_caster_wheel"/>
   <xacro:s40a_lb_lrf_mount_joint
-    name="front_lrf_mount"
+    name="front_lrf_mount_joint"
     xyz="0.0 0.0 0.0" rpy="0 0 ${radians(0)}"
     parent="body_link"
     child="front_lrf_mount"/>
   <xacro:s40a_lb_lrf_mount_joint
-    name="back_lrf_mount"
+    name="back_lrf_mount_joint"
     xyz="0.0 0.0 0.0" rpy="0 0 ${radians(180)}"
     parent="body_link"
     child="back_lrf_mount"/>
+  <xacro:gazebo_sensors />
 </robot>

File: urdf/s40a_lb_ros2_control.xacro (robot description, xacro)
@@ -3,5 +3,5 @@
   <ros2_control name="GazeboSystem" type="system">
     <hardware>
-      <plugin>gazebo_ros2_control/GazeboSystem</plugin>
+      <plugin>gz_ros2_control/GazeboSimSystem</plugin>
     </hardware>
     <joint name="left_wheel_joint">
@@ -39,20 +39,4 @@
       <state_interface name="velocity"/>
     </joint>
-    <joint name="front_left_caster_steering_joint">
-      <state_interface name="position"/>
-      <state_interface name="velocity"/>
-    </joint>
-    <joint name="front_right_caster_steering_joint">
-      <state_interface name="position"/>
-      <state_interface name="velocity"/>
-    </joint>
-    <joint name="back_right_caster_steering_joint">
-      <state_interface name="position"/>
-      <state_interface name="velocity"/>
-    </joint>
-    <joint name="back_left_caster_steering_joint">
-      <state_interface name="position"/>
-      <state_interface name="velocity"/>
-    </joint>
     <joint name="front_left_caster_wheel_joint">
       <state_interface name="position"/>

Commit message: Use native URDF tire contacts and remove custom friction system

File: urdf/f120a.xacro (robot description, xacro)
@@ -162,7 +162,19 @@
     </visual>
     <collision>
-      <origin xyz="-0.108 0.197 -0.085" rpy="0 0 0" />
-      <geometry>
-        <mesh filename="package://megarover_description/meshes/f120a/right_wheel_1.stl" scale="0.001 0.001 0.001" />
+      <origin xyz="0 -0.015 0" rpy="1.5708 0 0"/>
+      <geometry>
+        <cylinder radius="0.085" length="0.015"/>
+      </geometry>
+    </collision>
+    <collision>
+      <origin xyz="0 0 0" rpy="1.5708 0 0"/>
+      <geometry>
+        <cylinder radius="0.085" length="0.015"/>
+      </geometry>
+    </collision>
+    <collision>
+      <origin xyz="0 0.015 0" rpy="1.5708 0 0"/>
+      <geometry>
+        <cylinder radius="0.085" length="0.015"/>
       </geometry>
     </collision>
@@ -190,7 +202,19 @@
     </visual>
     <collision>
-      <origin xyz="-0.108297 -0.202941 -0.087693" rpy="0 0 0" />
-      <geometry>
-        <mesh filename="package://megarover_description/meshes/f120a/left_wheel_1.stl" scale="0.001 0.001 0.001" />
+      <origin xyz="0 -0.015 0" rpy="1.5708 0 0"/>
+      <geometry>
+        <cylinder radius="0.085" length="0.015"/>
+      </geometry>
+    </collision>
+    <collision>
+      <origin xyz="0 0 0" rpy="1.5708 0 0"/>
+      <geometry>
+        <cylinder radius="0.085" length="0.015"/>
+      </geometry>
+    </collision>
+    <collision>
+      <origin xyz="0 0.015 0" rpy="1.5708 0 0"/>
+      <geometry>
+        <cylinder radius="0.085" length="0.015"/>
       </geometry>
     </collision>

File: urdf/mega3.xacro (robot description, xacro)
@@ -163,7 +163,25 @@
     </visual>
     <collision>
-      <origin xyz="-0.1 -0.136 -0.07" rpy="0 0 -1.5708" />
-      <geometry>
-        <mesh filename="package://megarover_description/meshes/mega3/left_wheel_1.stl" scale="0.001 0.001 0.001" />
+      <origin xyz="0 0 0" rpy="-1.5708 0 0"/>
+      <geometry>
+        <cylinder radius="0.069965" length="0.006227"/>
+      </geometry>
+    </collision>
+    <collision>
+      <origin xyz="0 0 0" rpy="-1.5708 0 0"/>
+      <geometry>
+        <cylinder radius="0.069687" length="0.018681"/>
+      </geometry>
+    </collision>
+    <collision>
+      <origin xyz="0 0 0" rpy="-1.5708 0 0"/>
+      <geometry>
+        <cylinder radius="0.069132" length="0.031134"/>
+      </geometry>
+    </collision>
+    <collision>
+      <origin xyz="0 0 0" rpy="-1.5708 0 0"/>
+      <geometry>
+        <cylinder radius="0.068300" length="0.043500"/>
       </geometry>
     </collision>
@@ -191,7 +209,25 @@
     </visual>
     <collision>
-      <origin xyz="-0.1 0.136 -0.07" rpy="0 0 -1.5708" />
-      <geometry>
-        <mesh filename="package://megarover_description/meshes/mega3/right_wheel_1.stl" scale="0.001 0.001 0.001" />
+      <origin xyz="0 0 0" rpy="-1.5708 0 0"/>
+      <geometry>
+        <cylinder radius="0.069965" length="0.006227"/>
+      </geometry>
+    </collision>
+    <collision>
+      <origin xyz="0 0 0" rpy="-1.5708 0 0"/>
+      <geometry>
+        <cylinder radius="0.069687" length="0.018681"/>
+      </geometry>
+    </collision>
+    <collision>
+      <origin xyz="0 0 0" rpy="-1.5708 0 0"/>
+      <geometry>
+        <cylinder radius="0.069132" length="0.031134"/>
+      </geometry>
+    </collision>
+    <collision>
+      <origin xyz="0 0 0" rpy="-1.5708 0 0"/>
+      <geometry>
+        <cylinder radius="0.068300" length="0.043500"/>
       </geometry>
     </collision>

File: urdf/s40a_lb.xacro (robot description, xacro)
@@ -51,7 +51,25 @@
     </visual>
     <collision>
-      <geometry>
-        <mesh filename="package://megarover_description/meshes/s40a_lb/wheel.stl"
-              scale="0.001 0.001 0.001"/>
+      <origin xyz="0 0 0.02885" rpy="0 0 0"/>
+      <geometry>
+        <cylinder radius="0.070000" length="0.001000"/>
+      </geometry>
+    </collision>
+    <collision>
+      <origin xyz="0 0 0.02885" rpy="0 0 0"/>
+      <geometry>
+        <cylinder radius="0.069811" length="0.014534"/>
+      </geometry>
+    </collision>
+    <collision>
+      <origin xyz="0 0 0.02885" rpy="0 0 0"/>
+      <geometry>
+        <cylinder radius="0.069244" length="0.029066"/>
+      </geometry>
+    </collision>
+    <collision>
+      <origin xyz="0 0 0.02885" rpy="0 0 0"/>
+      <geometry>
+        <cylinder radius="0.068300" length="0.043500"/>
       </geometry>
     </collision>
@@ -120,7 +138,7 @@
     </visual>
     <collision>
-      <geometry>
-        <mesh filename="package://megarover_description/meshes/s40a_lb/caster_wheel.stl"
-              scale="0.001 0.001 0.001"/>
+      <origin xyz="0 0 0.01"/>
+      <geometry>
+        <cylinder radius="0.0325" length="0.02"/>
       </geometry>
     </collision>
