Commit message: Align native joint limits and S40 suspension with supplied Isaac models

File: urdf/f120a.xacro (robot description, xacro)
@@ -145,4 +145,5 @@
     <child link="right_wheel_1" />
     <axis xyz="0.0 1.0 0.0" />
+    <limit effort="18.0" velocity="26.180" />
   </joint>
   <link name="right_wheel_1">
@@ -185,4 +186,5 @@
     <child link="left_wheel_1" />
     <axis xyz="0.0 1.0 0.0" />
+    <limit effort="18.0" velocity="26.180" />
   </joint>
   <link name="left_wheel_1">

File: urdf/mega3.xacro (robot description, xacro)
@@ -146,4 +146,5 @@
     <child link="left_wheel_1" />
     <axis xyz="0.0 1.0 0.0" />
+    <limit effort="3.5" velocity="28.274" />
   </joint>
   <link name="left_wheel_1">
@@ -192,4 +193,5 @@
     <child link="right_wheel_1" />
     <axis xyz="0.0 1.0 0.0" />
+    <limit effort="3.5" velocity="28.274" />
   </joint>
   <link name="right_wheel_1">

File: urdf/s40a_lb.xacro (robot description, xacro)
@@ -241,6 +241,6 @@
       <child link="${child}"/>
       <axis xyz="0 0 -1"/>
-      <limit lower="-0.015" upper="0.006" effort="100" velocity="20.0"/>
-      <dynamics damping="280.0" friction="0.0"/>
+      <limit lower="0.0" upper="0.0135" effort="451.2" velocity="20.0"/>
+      <dynamics damping="1000.0" friction="0.0"/>
     </joint>
   </xacro:macro>
@@ -252,5 +252,5 @@
       <child link="${child}"/>
       <axis xyz="0 0 ${axis_z}"/>
-      <limit effort="500" velocity="50000"/>
+      <limit effort="3.5" velocity="28.274"/>
       <dynamics damping="0.02"/>
     </joint>
@@ -263,6 +263,6 @@
       <child link="${child}"/>
       <axis xyz="0 0 -1"/>
-      <limit lower="-0.015" upper="0.006" effort="1000" velocity="20.0"/>
-      <dynamics damping="120.0" friction="0.0"/>
+      <limit lower="0.0" upper="0.0135" effort="392.3" velocity="20.0"/>
+      <dynamics damping="1000.0" friction="0.0"/>
     </joint>
   </xacro:macro>

Commit message: Publish verified ROS 2 Jazzy and Gazebo Harmonic package
Import the qualified package files and use the public Jazzy clone URLs.

File: urdf/f120a.xacro (robot description, xacro)
@@ -145,5 +145,4 @@
     <child link="right_wheel_1" />
     <axis xyz="0.0 1.0 0.0" />
-    <limit effort="18.0" velocity="26.180" />
   </joint>
   <link name="right_wheel_1">
@@ -163,19 +162,7 @@
     </visual>
     <collision>
-      <origin xyz="0 -0.015 0" rpy="1.5708 0 0"/>
+      <origin xyz="-0.108 0.197 -0.085" rpy="0 0 0" />
       <geometry>
-        <cylinder radius="0.085" length="0.015"/>
-      </geometry>
-    </collision>
-    <collision>
-      <origin xyz="0 0 0" rpy="1.5708 0 0"/>
-      <geometry>
-        <cylinder radius="0.085" length="0.015"/>
-      </geometry>
-    </collision>
-    <collision>
-      <origin xyz="0 0.015 0" rpy="1.5708 0 0"/>
-      <geometry>
-        <cylinder radius="0.085" length="0.015"/>
+        <mesh filename="package://megarover_description/meshes/f120a/right_wheel_1.stl" scale="0.001 0.001 0.001" />
       </geometry>
     </collision>
@@ -186,5 +173,4 @@
     <child link="left_wheel_1" />
     <axis xyz="0.0 1.0 0.0" />
-    <limit effort="18.0" velocity="26.180" />
   </joint>
   <link name="left_wheel_1">
@@ -204,19 +190,7 @@
     </visual>
     <collision>
-      <origin xyz="0 -0.015 0" rpy="1.5708 0 0"/>
+      <origin xyz="-0.108297 -0.202941 -0.087693" rpy="0 0 0" />
       <geometry>
-        <cylinder radius="0.085" length="0.015"/>
-      </geometry>
-    </collision>
-    <collision>
-      <origin xyz="0 0 0" rpy="1.5708 0 0"/>
-      <geometry>
-        <cylinder radius="0.085" length="0.015"/>
-      </geometry>
-    </collision>
-    <collision>
-      <origin xyz="0 0.015 0" rpy="1.5708 0 0"/>
-      <geometry>
-        <cylinder radius="0.085" length="0.015"/>
+        <mesh filename="package://megarover_description/meshes/f120a/left_wheel_1.stl" scale="0.001 0.001 0.001" />
       </geometry>
     </collision>

File: urdf/mega3.xacro (robot description, xacro)
@@ -12,7 +12,5 @@
   <!-- <xacro:include filename="$(find vs_rover_options_description)/urdf/lrf/tg30_mega3.xacro" /> -->
   <!-- OPTION  bumper sensor -->
-  <!-- <xacro:include filename="$(find vs_rover_options_description)/urdf/bumper/bumper_mega3.xacro" />
-  <xacro:bumperbaseboard prefix="front" parent="base_link" xyz="0.19 0 0.02" z_dir="90" />
-  <xacro:bumperbaseboard prefix="back" parent="base_link" xyz="-0.19 0 0.02" z_dir="-90" />-->
+  <!-- <xacro:include filename="$(find vs_rover_options_description)/urdf/bumper/bumper_mega3.xacro" /> -->
   <!-- OPTION  camera stay -->
   <!-- <xacro:include filename="$(find vs_rover_options_description)/urdf/cam_stay/cam_stay_mega3.xacro" />
@@ -146,5 +144,4 @@
     <child link="left_wheel_1" />
     <axis xyz="0.0 1.0 0.0" />
-    <limit effort="3.5" velocity="28.274" />
   </joint>
   <link name="left_wheel_1">
@@ -164,25 +161,7 @@
     </visual>
     <collision>
-      <origin xyz="0 0 0" rpy="-1.5708 0 0"/>
+      <origin xyz="-0.1 -0.136 -0.07" rpy="0 0 -1.5708" />
       <geometry>
-        <cylinder radius="0.069965" length="0.006227"/>
-      </geometry>
-    </collision>
-    <collision>
-      <origin xyz="0 0 0" rpy="-1.5708 0 0"/>
-      <geometry>
-        <cylinder radius="0.069687" length="0.018681"/>
-      </geometry>
-    </collision>
-    <collision>
-      <origin xyz="0 0 0" rpy="-1.5708 0 0"/>
-      <geometry>
-        <cylinder radius="0.069132" length="0.031134"/>
-      </geometry>
-    </collision>
-    <collision>
-      <origin xyz="0 0 0" rpy="-1.5708 0 0"/>
-      <geometry>
-        <cylinder radius="0.068300" length="0.043500"/>
+        <mesh filename="package://megarover_description/meshes/mega3/left_wheel_1.stl" scale="0.001 0.001 0.001" />
       </geometry>
     </collision>
@@ -193,5 +172,4 @@
     <child link="right_wheel_1" />
     <axis xyz="0.0 1.0 0.0" />
-    <limit effort="3.5" velocity="28.274" />
   </joint>
   <link name="right_wheel_1">
@@ -211,25 +189,7 @@
     </visual>
     <collision>
-      <origin xyz="0 0 0" rpy="-1.5708 0 0"/>
+      <origin xyz="-0.1 0.136 -0.07" rpy="0 0 -1.5708" />
       <geometry>
-        <cylinder radius="0.069965" length="0.006227"/>
-      </geometry>
-    </collision>
-    <collision>
-      <origin xyz="0 0 0" rpy="-1.5708 0 0"/>
-      <geometry>
-        <cylinder radius="0.069687" length="0.018681"/>
-      </geometry>
-    </collision>
-    <collision>
-      <origin xyz="0 0 0" rpy="-1.5708 0 0"/>
-      <geometry>
-        <cylinder radius="0.069132" length="0.031134"/>
-      </geometry>
-    </collision>
-    <collision>
-      <origin xyz="0 0 0" rpy="-1.5708 0 0"/>
-      <geometry>
-        <cylinder radius="0.068300" length="0.043500"/>
+        <mesh filename="package://megarover_description/meshes/mega3/right_wheel_1.stl" scale="0.001 0.001 0.001" />
       </geometry>
     </collision>

File: urdf/s40a_lb.xacro (robot description, xacro)
@@ -51,25 +51,7 @@
     </visual>
     <collision>
-      <origin xyz="0 0 0.02885" rpy="0 0 0"/>
-      <geometry>
-        <cylinder radius="0.070000" length="0.001000"/>
-      </geometry>
-    </collision>
-    <collision>
-      <origin xyz="0 0 0.02885" rpy="0 0 0"/>
-      <geometry>
-        <cylinder radius="0.069811" length="0.014534"/>
-      </geometry>
-    </collision>
-    <collision>
-      <origin xyz="0 0 0.02885" rpy="0 0 0"/>
-      <geometry>
-        <cylinder radius="0.069244" length="0.029066"/>
-      </geometry>
-    </collision>
-    <collision>
-      <origin xyz="0 0 0.02885" rpy="0 0 0"/>
-      <geometry>
-        <cylinder radius="0.068300" length="0.043500"/>
+      <geometry>
+        <mesh filename="package://megarover_description/meshes/s40a_lb/wheel.stl"
+              scale="0.001 0.001 0.001"/>
       </geometry>
     </collision>
@@ -138,7 +120,7 @@
     </visual>
     <collision>
-      <origin xyz="0 0 0.01"/>
-      <geometry>
-        <cylinder radius="0.0325" length="0.02"/>
+      <geometry>
+        <mesh filename="package://megarover_description/meshes/s40a_lb/caster_wheel.stl"
+              scale="0.001 0.001 0.001"/>
       </geometry>
     </collision>
@@ -241,6 +223,6 @@
       <child link="${child}"/>
       <axis xyz="0 0 -1"/>
-      <limit lower="0.0" upper="0.0135" effort="451.2" velocity="20.0"/>
-      <dynamics damping="1000.0" friction="0.0"/>
+      <limit lower="-0.015" upper="0.006" effort="100" velocity="20.0"/>
+      <dynamics damping="280.0" friction="0.0"/>
     </joint>
   </xacro:macro>
@@ -252,5 +234,5 @@
       <child link="${child}"/>
       <axis xyz="0 0 ${axis_z}"/>
-      <limit effort="3.5" velocity="28.274"/>
+      <limit effort="500" velocity="50000"/>
       <dynamics damping="0.02"/>
     </joint>
@@ -263,6 +245,6 @@
       <child link="${child}"/>
       <axis xyz="0 0 -1"/>
-      <limit lower="0.0" upper="0.0135" effort="392.3" velocity="20.0"/>
-      <dynamics damping="1.0" friction="0.0"/>
+      <limit lower="-0.015" upper="0.006" effort="1000" velocity="20.0"/>
+      <dynamics damping="120.0" friction="0.0"/>
     </joint>
   </xacro:macro>
