Commit message: Correct native S40 caster damping at the suspension travel limit

File: urdf/s40a_lb.xacro (robot description, xacro)
@@ -264,5 +264,5 @@
       <axis xyz="0 0 -1"/>
       <limit lower="0.0" upper="0.0135" effort="392.3" velocity="20.0"/>
-      <dynamics damping="1000.0" friction="0.0"/>
+      <dynamics damping="1.0" friction="0.0"/>
     </joint>
   </xacro:macro>
